File: Aviônica/Aviônica 3.0 - Para corrosão/esquema.brd (EAGLE design)
At the start: 115 x 75.1 mm, 15 parts, among them M1 WIRELESS-NRF24L01-PA-EXT

Commit message: Update
Routing:
- net 3V3_2: track 5.66 -> 0.00 mm
Changed lines of the file:
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@@
 <wire x1="-0.03" y1="-1.98" x2="-0.03" y2="73.11" width="0" layer="20"/>
 <wire x1="114.97" y1="-1.89" x2="0" y2="-1.99" width="0" layer="20"/>
-<dimension x1="112" y1="106" x2="7" y2="106" x3="59.5" y3="108" textsize="1.778" layer="20"/>
 </plain>
 <attributes>
@@
 <contactref element="U$4" pad="3V3_2"/>
 <contactref element="JP5" pad="1"/>
-<wire x1="19" y1="4" x2="15" y2="8" width="1" layer="1"/>
 <wire x1="34.77" y1="9.57" x2="96.89" y2="5.525" width="0" layer="19" extent="1-1"/>
-<wire x1="19" y1="4" x2="34.77" y2="9.57" width="0" layer="19" extent="1-1"/>
-<wire x1="18" y1="49" x2="15" y2="8" width="0" layer="19" extent="1-1"/>
+<wire x1="18" y1="49" x2="34.77" y2="9.57" width="0" layer="19" extent="1-1"/>
 </signal>
 <signal name="CE">
