File: Paraquedas/Paraquedas 2.0 - 2 skibs - Para corrosão/Esquema.brd (EAGLE design)
At the start: 51 x 57 mm, 13 parts, among them Q1 IRF540, Q2 IRF540, Q3 IRF540

Commit message: Atualizando placas
Parts:
- moved R1 37.0 mm to (43.0, 26.0), flipped to the bottom
- moved E4 31.6 mm to (8.70, 3.80), flipped to the bottom
- moved Q2 29.6 mm to (9.69, 21.1), flipped to the bottom
- moved SKIB2 29.6 mm to (9.69, 45.2), flipped to the bottom
- moved E3 26.0 mm to (11.5, 3.80), flipped to the bottom
- moved Q3 21.0 mm to (35.0, 21.0), flipped to the bottom
- moved SP2 21.0 mm to (35.0, 44.0), flipped to the bottom
- moved BATERIA 20.9 mm to (35.0, 4.84), flipped to the bottom
- moved E2 20.5 mm to (14.3, 3.83), flipped to the bottom
- moved E5 15.0 mm to (17.0, 3.80), flipped to the bottom
- moved E1 9.52 mm to (19.7, 3.83), flipped to the bottom
- moved Q1 4.22 mm to (22.4, 21.1), flipped to the bottom
- moved SKIB1 4.22 mm to (22.4, 45.2), flipped to the bottom
Routing:
- added copper zone on layer 16, net GND
- removed copper zone on layer 1, net GND

Commit message: Update
Parts:
- moved E5 2.88 mm to (14.1, 3.78)
- moved E2 2.57 mm to (16.8, 3.79)
- moved E4 2.40 mm to (6.30, 3.80)
- moved E1 0.20 mm to (19.6, 3.78)
- moved E3 0.10 mm to (11.4, 3.80)
Routing:
- net GND: track 5.00 -> 0.00 mm, vias 2 -> 0
- net SKIB1: track 20.9 -> 17.3 mm
- net N$4: track 13.9 -> 15.6 mm
- net VCC: track 85.7 -> 86.8 mm
- net BUZZER: track 42.1 -> 43.1 mm
- net S1: track 33.6 -> 34.6 mm
- net S2: track 33.6 -> 34.5 mm
- added copper zone on layer 16, net DS
