File: Paraquedas/Paraquedas 2.1 - 2 skibs - Para corrosão/Esquema.brd (EAGLE design)
At the start: 51 x 57 mm, 13 parts, among them Q1 IRF540, Q2 IRF540, Q3 IRF540

Commit message: Message
Other:
- board size 51 x 57 mm -> 51.5 x 57 mm
Changed lines of the file:
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@@
 <layers>
 <layer number="1" name="Top" color="4" fill="1" visible="yes" active="yes"/>
-<layer number="2" name="Route2" color="16" fill="1" visible="yes" active="yes"/>
+<layer number="2" name="Route2" color="16" fill="1" visible="no" active="no"/>
 <layer number="3" name="Route3" color="17" fill="1" visible="no" active="no"/>
 <layer number="4" name="Route4" color="18" fill="1" visible="no" active="no"/>
@@
 <layer number="13" name="Route13" color="21" fill="1" visible="no" active="no"/>
 <layer number="14" name="Route14" color="22" fill="1" visible="no" active="no"/>
-<layer number="15" name="Route15" color="23" fill="1" visible="yes" active="yes"/>
+<layer number="15" name="Route15" color="23" fill="1" visible="no" active="no"/>
 <layer number="16" name="Bottom" color="1" fill="1" visible="yes" active="yes"/>
 <layer number="17" name="Pads" color="2" fill="1" visible="yes" active="yes"/>
@@
 </layers>
 <board>
-<fusionsync huburn="a.YnVzaW5lc3M6ZGlzY2VudGU3MA" projecturn="a.YnVzaW5lc3M6ZGlzY2VudGU3MCMyMDIyMDIxNzQ5ODU5MDQ4MQ" f3durn="urn:adsk.wipprod:dm.lineage:eC2E5IMDRm2aw-eJDvErbw" pcbguid="" lastpulledtime="" lastsyncedchangeguid="" latestrevisionid="d5523bd2-7437-4db2-b767-71d2d1ac56fe" lastsyncedrevisionid="d5523bd2-7437-4db2-b767-71d2d1ac56fe" lastboardhashguid="33d128af-a64a-b0db-033b-a1b71b82984a" lastpushedtime="2023-05-09T12:36:54Z" linktopcb3d="true"/>
+<fusionsync huburn="a.YnVzaW5lc3M6ZGlzY2VudGU3MA" projecturn="a.YnVzaW5lc3M6ZGlzY2VudGU3MCMyMDIyMDIxNzQ5ODU5MDQ4MQ" f3durn="urn:adsk.wipprod:dm.lineage:eC2E5IMDRm2aw-eJDvErbw" pcbguid="" lastpulledtime="" lastsyncedchangeguid="" latestrevisionid="d5523bd2-7437-4db2-b767-71d2d1ac56fe" lastsyncedrevisionid="d5523bd2-7437-4db2-b767-71d2d1ac56fe" lastboardhashguid="33d128af-a64a-b0db-033b-a1b71b82984a" lastpushedtime="2023-05-09T12:36:54Z" linktopcb3d="false"/>
 <plain>
-<wire x1="50" y1="-3" x2="-1" y2="-3" width="0" layer="20"/>
+<wire x1="50.5" y1="-3" x2="-1" y2="-3" width="0" layer="20"/>
 <wire x1="-1" y1="-3" x2="-1" y2="54" width="0" layer="20"/>
-<wire x1="-1" y1="54" x2="50" y2="54" width="0" layer="20"/>
-<wire x1="50" y1="54" x2="50" y2="-3" width="0" layer="20"/>
+<wire x1="-1" y1="54" x2="50.5" y2="54" width="0" layer="20"/>
+<wire x1="50.5" y1="54" x2="50.5" y2="-3" width="0" layer="20"/>
 <dimension x1="-1" y1="-5" x2="50" y2="-5" x3="24.5" y3="-9" textsize="1.778" layer="20"/>
 <dimension x1="-5" y1="-3" x2="-5" y2="54" x3="-9" y3="25.5" textsize="1.778" layer="20"/>
 <hole x="2" y="51" drill="3"/>
-<hole x="47" y="51" drill="3"/>
+<hole x="47.5" y="51" drill="3"/>
 <hole x="2" y="0" drill="3"/>
-<hole x="47" y="0" drill="3"/>
+<hole x="47.6" y="0" drill="3"/>
 </plain>
 <attributes>
@@
 necessary adjustments and save your customized
 design rules under a new name.</description>
-<param name="layerSetup" value="(1*2+15*16)"/>
+<param name="layerSetup" value="(1*16)"/>
 <param name="mtCopper" value="0.035mm 0.035mm 0.035mm 0.035mm 0.035mm 0.035mm 0.035mm 0.035mm 0.035mm 0.035mm 0.035mm 0.035mm 0.035mm 0.035mm 0.035mm 0.035mm"/>
 <param name="mtIsolate" value="1.5mm 0.15mm 0.2mm 0.15mm 0.2mm 0.15mm 0.2mm 0.15mm 0.2mm 0.15mm 0.2mm 0.15mm 0.2mm 0.15mm 0.2mm"/>
-<param name="mdWireWire" value="30mil"/>
-<param name="mdWirePad" value="0.5mm"/>
-<param name="mdWireVia" value="6mil"/>
-<param name="mdPadPad" value="6mil"/>
-<param name="mdPadVia" value="6mil"/>
-<param name="mdViaVia" value="6mil"/>
+<param name="mdWireWire" value="40mil"/>
+<param name="mdWirePad" value="10mil"/>
+<param name="mdWireVia" value="10mil"/>
+<param name="mdPadPad" value="10mil"/>
+<param name="mdPadVia" value="10mil"/>
+<param name="mdViaVia" value="10mil"/>
 <param name="mdSmdPad" value="6mil"/>
 <param name="mdSmdVia" value="6mil"/>
@@
 <contactref element="Q3" pad="1"/>
 <wire x1="42.7" y1="3.8" x2="42.7" y2="2.8" width="1" layer="16"/>
-<wire x1="42.7" y1="2.8" x2="39.9" y2="0" width="1" layer="16"/>
-<wire x1="39.9" y1="0" x2="23" y2="0" width="1" layer="16"/>
+<wire x1="42.7" y1="2.8" x2="39.4" y2="-0.5" width="1" layer="16"/>
+<wire x1="39.4" y1="-0.5" x2="23.5" y2="-0.5" width="1" layer="16"/>
 <wire x1="21" y1="2" x2="21" y2="8" width="1" layer="16"/>
 <wire x1="21" y1="8" x2="17.0264" y2="11.9736" width="1" layer="16"/>
@@
 <wire x1="13" y1="12" x2="11.46" y2="13.54" width="1" layer="16"/>
 <wire x1="11.46" y1="13.54" x2="11.46" y2="14.65" width="1" layer="16"/>
-<wire x1="23" y1="0" x2="21" y2="2" width="1" layer="16"/>
+<wire x1="23.5" y1="-0.5" x2="21" y2="2" width="1" layer="16"/>
 </signal>
 <signal name="GND">
@@
 <contactref element="Q3" pad="3"/>
 <polygon width="1.016" layer="16" orphans="yes">
-<vertex x="49" y="53"/>
-<vertex x="49" y="-2"/>
+<vertex x="50" y="53"/>
+<vertex x="50" y="-2"/>
 <vertex x="0" y="-2"/>
 <vertex x="0" y="53"/>
@@
 <wire x1="16.714" y1="49" x2="20.2954" y2="49" width="1" layer="16"/>
 <wire x1="16.5546" y1="4.84" x2="16.5546" y2="7.4454" width="1" layer="16"/>
-<wire x1="14" y1="10" x2="5" y2="10" width="1" layer="16"/>
-<wire x1="16.5546" y1="7.4454" x2="14" y2="10" width="1" layer="16"/>
-<wire x1="5" y1="10" x2="2.857" y2="12.143" width="1" layer="16"/>
+<wire x1="14.4" y1="9.6" x2="5.4" y2="9.6" width="1" layer="16"/>
+<wire x1="16.5546" y1="7.4454" x2="14.4" y2="9.6" width="1" layer="16"/>
+<wire x1="5.4" y1="9.6" x2="2.857" y2="12.143" width="1" layer="16"/>
 <wire x1="2.857" y1="12.143" x2="2.857" y2="37.143" width="1" layer="16"/>
 </signal>
