File: Aviônica/Aviônica 2.1 - Para corrosão/esquema.brd (EAGLE design)
At the start: 129 x 66 mm, 15 parts, among them M1 WIRELESS-NRF24L01-PA-EXT

Commit message: Upgrage
Routing:
- net 3V3_2: track 195.2 -> 195.8 mm
- net 3V3_1: track 90.2 -> 90.7 mm
Changed lines of the file:
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@@
 <element name="U$5" library="CRD" library_urn="urn:adsk.eagle:library:39051337" package="JST2.54X2P_FOOTPRINT" package3d_urn="urn:adsk.eagle:package:39191967/2" value="JST2.54X2P" x="6.54" y="10.11" smashed="yes" rot="R270"/>
 <element name="U$6" library="CRD" library_urn="urn:adsk.eagle:library:39051337" package="SWITCH_3PIN" package3d_urn="urn:adsk.eagle:package:39192263/6" value="SWITCH_3PIN" x="6.7" y="22.1" smashed="yes" rot="R90"/>
-<element name="U$4" library="CRD" library_urn="urn:adsk.eagle:library:39051337" package="WIFI_KIT32" package3d_urn="urn:adsk.eagle:package:39051622/7" value="WIFI_KIT32" x="67.2" y="18.3" smashed="yes" rot="R90"/>
+<element name="U$4" library="CRD" library_urn="urn:adsk.eagle:library:39051337" package="WIFI_KIT32" package3d_urn="urn:adsk.eagle:package:39051622/9" value="WIFI_KIT32" x="67.2" y="18.3" smashed="yes" rot="R90"/>
 <element name="JP1" library="pinhead" library_urn="urn:adsk.eagle:library:325" package="1X01" package3d_urn="urn:adsk.eagle:package:22485/2" value="SKIB1" x="14.4" y="58" smashed="yes">
 <attribute name="NAME" x="13.0538" y="59.8288" size="1.27" layer="25" ratio="10"/>
@@
 <wire x1="32" y1="30" x2="35" y2="27" width="1" layer="16"/>
 <wire x1="58" y1="27" x2="59.28" y2="28.28" width="1" layer="16"/>
-<wire x1="59.28" y1="28.28" x2="59.28" y2="29.638" width="1" layer="16"/>
+<wire x1="59.28" y1="28.28" x2="58.31" y2="29.73" width="1" layer="16"/>
 </signal>
 <signal name="SDA">
@@
 <wire x1="23.4055" y1="12.5945" x2="26.87" y2="12.5945" width="1" layer="16"/>
 <wire x1="33.9945" y1="12.5945" x2="26.87" y2="12.5945" width="1" layer="16"/>
-<wire x1="35.52" y1="6.905" x2="35.52" y2="11.069" width="1" layer="16"/>
+<wire x1="35.45" y1="6.87" x2="35.52" y2="11.069" width="1" layer="16"/>
 <wire x1="35.52" y1="11.069" x2="33.9945" y2="12.5945" width="1" layer="16"/>
 </signal>
@@
 <wire x1="97" y1="28.08" x2="97" y2="30.9" width="1" layer="16"/>
 <wire x1="97" y1="30.9" x2="97.1" y2="31" width="1" layer="16"/>
-<wire x1="56.64" y1="29.638" x2="56.64" y2="32.624" width="1" layer="16"/>
+<wire x1="55.77" y1="29.73" x2="56.64" y2="32.624" width="1" layer="16"/>
 <wire x1="56.64" y1="32.624" x2="58" y2="33.984" width="1" layer="16"/>
 </signal>
@@
 <contactref element="R2" pad="2"/>
 <wire x1="101" y1="28.08" x2="101" y2="30" width="1" layer="16"/>
-<wire x1="54" y1="29.638" x2="54" y2="33" width="1" layer="16"/>
+<wire x1="53.23" y1="29.73" x2="54" y2="33" width="1" layer="16"/>
 <wire x1="54" y1="33" x2="57" y2="36" width="1" layer="16"/>
 <wire x1="102.14894375" y1="36" x2="95" y2="36" width="1" layer="1"/>
@@
 <wire x1="88.148" y1="11.551" x2="89.731" y2="9.968" width="1" layer="16"/>
 <wire x1="89.731" y1="9.968" x2="102.968" y2="9.968" width="1" layer="16"/>
-<wire x1="48.72" y1="29.638" x2="48.72" y2="34.752" width="1" layer="16"/>
+<wire x1="48.15" y1="29.73" x2="48.72" y2="34.752" width="1" layer="16"/>
 <wire x1="48.72" y1="34.752" x2="54" y2="40.032" width="1" layer="16"/>
 </signal>
@@
 <wire x1="88.829" y1="14.171" x2="88.148" y2="14.171" width="1" layer="16"/>
 <wire x1="91.016" y1="11.984" x2="88.829" y2="14.171" width="1" layer="16"/>
-<wire x1="51.36" y1="29.638" x2="51.36" y2="33.376" width="1" layer="16"/>
+<wire x1="50.69" y1="29.73" x2="51.36" y2="33.376" width="1" layer="16"/>
 <wire x1="51.36" y1="33.376" x2="56" y2="38.016" width="1" layer="16"/>
 </signal>
@@
 <wire x1="15" y1="9" x2="15" y2="44" width="1" layer="16"/>
 <wire x1="47" y1="4" x2="74" y2="4" width="1" layer="16"/>
-<wire x1="75.12" y1="6.905" x2="75.12" y2="5.12" width="1" layer="16"/>
+<wire x1="73.55" y1="6.87" x2="75.12" y2="5.12" width="1" layer="16"/>
 <wire x1="75.12" y1="5.12" x2="74" y2="4" width="1" layer="16"/>
 <wire x1="110" y1="4" x2="76.24" y2="4" width="1" layer="16"/>
@@
 <wire x1="120" y1="41" x2="121.484" y2="42.484" width="1" layer="16"/>
 <wire x1="45" y1="1" x2="113" y2="1" width="1" layer="16"/>
-<wire x1="40.8" y1="6.905" x2="40.8" y2="5.2" width="1" layer="16"/>
+<wire x1="40.53" y1="6.87" x2="40.8" y2="5.2" width="1" layer="16"/>
 <wire x1="40.8" y1="5.2" x2="45" y2="1" width="1" layer="16"/>
 </signal>
@@
 <contactref element="U$4" pad="2"/>
 <wire x1="47" y1="48.73" x2="116.875" y2="48.73" width="1" layer="16"/>
-<wire x1="43.44" y1="29.638" x2="43.44" y2="45.17" width="1" layer="16"/>
+<wire x1="43.07" y1="29.73" x2="43.44" y2="45.17" width="1" layer="16"/>
 <wire x1="43.44" y1="45.17" x2="47" y2="48.73" width="1" layer="16"/>
 </signal>
@@
 <wire x1="32" y1="47" x2="17" y2="47" width="1" layer="16"/>
 <wire x1="17" y1="47" x2="14.4" y2="49.6" width="1" layer="16"/>
-<wire x1="35.52" y1="29.638" x2="35.52" y2="43.48" width="1" layer="16"/>
+<wire x1="35.45" y1="29.73" x2="35.52" y2="43.48" width="1" layer="16"/>
 <wire x1="35.52" y1="43.48" x2="32" y2="47" width="1" layer="16"/>
 </signal>
@@
 <contactref element="U$4" pad="17"/>
 <wire x1="32.83505625" y1="49.016" x2="19.884" y2="49.016" width="1" layer="16"/>
-<wire x1="38.16" y1="29.638" x2="38.16" y2="43.69105625" width="1" layer="16"/>
+<wire x1="37.99" y1="29.73" x2="38.16" y2="43.69105625" width="1" layer="16"/>
 <wire x1="38.16" y1="43.69105625" x2="32.83505625" y2="49.016" width="1" layer="16"/>
 <wire x1="17.1" y1="51.8" x2="17.1" y2="58" width="1" layer="16"/>
@@
 <contactref element="U$4" pad="4"/>
 <wire x1="19.8" y1="53" x2="19.8" y2="58" width="1" layer="16"/>
-<wire x1="40.8" y1="29.638" x2="40.8" y2="43.9021125" width="1" layer="16"/>
+<wire x1="40.53" y1="29.73" x2="40.8" y2="43.9021125" width="1" layer="16"/>
 <wire x1="40.8" y1="43.9021125" x2="40.07195" y2="44.6301625" width="1" layer="16"/>
 <wire x1="40.07195" y1="44.6301625" x2="39.52525625" y2="45.215346875" width="1" layer="16"/>
@@
 <wire x1="80.3" y1="22.3" x2="87.879" y2="22.3" width="1" layer="16"/>
 <wire x1="77.6323" y1="9.6323" x2="75.2646" y2="12" width="1" layer="16"/>
-<wire x1="77.76" y1="6.905" x2="77.76" y2="9.5046" width="1" layer="16"/>
+<wire x1="76.09" y1="6.87" x2="77.76" y2="9.5046" width="1" layer="16"/>
 <wire x1="77.6323" y1="9.6323" x2="77.76" y2="9.5046" width="1" layer="16"/>
 <wire x1="77.6323" y1="9.6323" x2="77.6323" y2="19.6323" width="1" layer="16"/>
