File: Solo/Solo 1.0/Esquemático.sch (EAGLE design)
At the start: 15 parts, among them M1 WIRELESS-NRF24L01-PA-EXT

Commit message: Message
Parts:
- removed JP1: SKIB1, pinhead:PINHD-1X1
- removed JP2: SKIB2, pinhead:PINHD-1X1
- removed JP3: BUZZER, pinhead:PINHD-1X1
- removed JP4: GND, pinhead:PINHD-1X1
- removed JP5: 3V3, pinhead:PINHD-1X1
- removed U$1: BMP280V1, CRD:BMP280V1
- removed U$2: MICROSD_READER, CRD:MICROSD_READER
- removed U$3: MPU6050V1, CRD:MPU6050V1
- removed U$4: WIFI_KIT32, CRD:WIFI_KIT32
- removed U$5, U$7: JST2.54X2P, CRD:JST2.54X2P
- removed U$6: SWITCH_3PIN, CRD:SWITCH_3PIN
- added ARDUINO_NANO1: (no value), ArduinoNanoV30:ARDUINO_NANO
- added LED1: (no value), led:LED5MM
- added S1: (no value), switch-omron:10-XX
- R1, R2: value 330 -> (none)
Connections:
- removed net 3V3_1: U$1.VCC, U$2.VCC, U$3.VCC, U$4.3V3_1
- removed net 3V3_2: JP5.1, M1.VCC, U$4.3V3_2
- removed net BUZZER: JP3.1, U$4.4
- removed net CE: M1.CE, U$4.12
- removed net CSN_NRF: M1.CSN, U$4.2
- removed net MISO: M1.MISO, R1.2, U$4.19
- removed net MISO_SD: R1.1, U$2.MISO
- removed net MOSI: M1.MOSI, R2.2, U$4.23
- removed net MOSI_SD: R2.1, U$2.MOSI
- removed net SCL: U$1.SCL, U$3.SCL, U$4.22
- removed net SCLK: M1.SCK, U$2.SCK, U$4.18
- removed net SDA: U$1.SDA, U$3.SDA, U$4.21
- removed net SKIB1: JP1.1, U$4.16
- removed net SKIB2: JP2.1, U$4.17
- removed net VIN: U$6.3, U$7.1
- removed net V_BATTERY: U$5.1, U$6.2
- new net N$10: ARDUINO_NANO1.3V3, M1.VCC
- new net N$2: ARDUINO_NANO1.D2, S1.P, S1.P1
- new net N$3: R2.2, S1.S, S1.S1
- new net N$4: ARDUINO_NANO1.D3, R1.1
- new net N$5: ARDUINO_NANO1.D13, M1.SCK
- new net N$6: ARDUINO_NANO1.D12, M1.MISO
- new net N$7: ARDUINO_NANO1.D11, M1.MOSI
- new net N$8: ARDUINO_NANO1.D7, M1.CE
- new net N$9: ARDUINO_NANO1.D8, M1.CSN
- net GND: now also ARDUINO_NANO1.GND@1, ARDUINO_NANO1.GND@2, LED1.C, R2.1; no longer JP4.1, U$1.GND, U$2.GND, U$3.GND, U$4.GND_1, U$4.GND_2, U$5.2, U$7.2
- net N$1: now also LED1.A, R1.2; no longer U$2.CS, U$4.5
Other:
- moved on the sheet: M1, R1, R2

Commit message: Upgrage
Changed lines of the file:
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@@
 <net name="N$10" class="0">
 <segment>
-<pinref part="M1" gate="G$1" pin="VCC"/>
-<wire x1="-86.36" y1="-27.94" x2="-50.8" y2="-27.94" width="0.1524" layer="91"/>
 <wire x1="-50.8" y1="-27.94" x2="-50.8" y2="-53.34" width="0.1524" layer="91"/>
 <wire x1="-50.8" y1="-53.34" x2="-2.54" y2="-53.34" width="0.1524" layer="91"/>
@@
 <wire x1="-2.54" y1="-53.34" x2="-2.54" y2="-20.32" width="0.1524" layer="91"/>
 <wire x1="-2.54" y1="-20.32" x2="-10.16" y2="-20.32" width="0.1524" layer="91"/>
+<pinref part="M1" gate="G$1" pin="VCC"/>
+<wire x1="-50.8" y1="-27.94" x2="-86.36" y2="-27.94" width="0.1524" layer="91"/>
 </segment>
 </net>
